File: touchdro-board/touchdro-board.kicad_pcb (KiCad board)
At the start: 2 copper layers, 3 parts, among them U1 74HC14, U2 74HC14, U3 ESP32_DevKit_V1_DOIT

Commit message: updates
Parts:
- removed U2: 74HC14, Package_DIP:DIP-14_W7.62mm
- added C1: 100n, Capacitor_THT:C_Rect_L7.2mm_W3.0mm_P5.00mm_FKS2_FKP2_MKS2_MKP2, F.Cu at (136.9, 59.4)
- added C10: 100n, Capacitor_THT:C_Rect_L7.2mm_W3.0mm_P5.00mm_FKS2_FKP2_MKS2_MKP2, F.Cu at (136.9, 91.8)
- added C11: 47u, Capacitor_THT:CP_Radial_D8.0mm_P3.50mm, F.Cu at (218.5, 110.6)
- added C2: 100n, Capacitor_THT:C_Rect_L7.2mm_W3.0mm_P5.00mm_FKS2_FKP2_MKS2_MKP2, F.Cu at (136.9, 63.5)
- added C4: 100n, Capacitor_THT:C_Rect_L7.2mm_W3.0mm_P5.00mm_FKS2_FKP2_MKS2_MKP2, F.Cu at (136.9, 71.6)
- added C5: 100n, Capacitor_THT:C_Rect_L7.2mm_W3.0mm_P5.00mm_FKS2_FKP2_MKS2_MKP2, F.Cu at (136.9, 75.6)
- added C6: 47u, Capacitor_THT:CP_Radial_D8.0mm_P3.50mm, F.Cu at (218.5, 101.0)
- added C7: 100n, Capacitor_THT:C_Rect_L7.2mm_W3.0mm_P5.00mm_FKS2_FKP2_MKS2_MKP2, F.Cu at (136.9, 79.7)
- added C8: 100n, Capacitor_THT:C_Rect_L7.2mm_W3.0mm_P5.00mm_FKS2_FKP2_MKS2_MKP2, F.Cu at (136.9, 83.7)
- added C9: 100n, Capacitor_THT:C_Rect_L7.2mm_W3.0mm_P5.00mm_FKS2_FKP2_MKS2_MKP2, F.Cu at (136.9, 87.8)
- added J1: USB_B_Micro, MicroUSB-Breakout:MicroUSB, F.Cu at (233.5, 56.7)
- added J2: USB_B_Micro, MicroUSB-Breakout:MicroUSB, F.Cu at (233.5, 71.1)
- added J3: Conn_01x03, Connector_PinHeader_2.54mm:PinHeader_1x03_P2.54mm_Vertical, F.Cu at (227.4, 105.8)
- added J4: USB_B_Micro, MicroUSB-Breakout:MicroUSB, F.Cu at (233.5, 85.5)
- added J5: Conn_01x03, Connector_PinHeader_2.54mm:PinHeader_1x03_P2.54mm_Vertical, F.Cu at (232.0, 105.8)
- added J6: Conn_01x03, Connector_PinHeader_2.54mm:PinHeader_1x03_P2.54mm_Vertical, F.Cu at (236.7, 105.8)
- added JP1: Jumper_2_Open, Connector_PinHeader_2.54mm:PinHeader_1x02_P2.54mm_Vertical, F.Cu at (227.4, 98.6)
- added JP2: Jumper_2_Open, Connector_PinHeader_2.54mm:PinHeader_1x02_P2.54mm_Vertical, F.Cu at (232.0, 98.6)
- added JP3: Jumper_2_Open, Connector_PinHeader_2.54mm:PinHeader_1x02_P2.54mm_Vertical, F.Cu at (236.7, 98.6)
- added R1: 4K7, Resistor_THT:R_Axial_DIN0207_L6.3mm_D2.5mm_P7.62mm_Horizontal, F.Cu at (203.5, 55.8)
- added R11: 47K, Resistor_THT:R_Axial_DIN0207_L6.3mm_D2.5mm_P7.62mm_Horizontal, F.Cu at (203.5, 78.0)
- added R12: 47K, Resistor_THT:R_Axial_DIN0207_L6.3mm_D2.5mm_P7.62mm_Horizontal, F.Cu at (203.5, 83.5)
- added R13: 47K, Resistor_THT:R_Axial_DIN0207_L6.3mm_D2.5mm_P7.62mm_Horizontal, F.Cu at (203.5, 89.0)
- added R14: 47K, Resistor_THT:R_Axial_DIN0207_L6.3mm_D2.5mm_P7.62mm_Horizontal, F.Cu at (203.5, 94.6)
- added R15: 4K7, Resistor_THT:R_Axial_DIN0207_L6.3mm_D2.5mm_P7.62mm_Horizontal, F.Cu at (203.5, 100.2)
- added R16: 4K7, Resistor_THT:R_Axial_DIN0207_L6.3mm_D2.5mm_P7.62mm_Horizontal, F.Cu at (203.5, 105.7)
- added R17: 47K, Resistor_THT:R_Axial_DIN0207_L6.3mm_D2.5mm_P7.62mm_Horizontal, F.Cu at (203.5, 111.2)
- added R18: 47K, Resistor_THT:R_Axial_DIN0207_L6.3mm_D2.5mm_P7.62mm_Horizontal, F.Cu at (203.5, 116.8)
- added R19: 4K7, Resistor_THT:R_Axial_DIN0207_L6.3mm_D2.5mm_P7.62mm_Horizontal, F.Cu at (203.5, 122.3)
- added R2: 4K7, Resistor_THT:R_Axial_DIN0207_L6.3mm_D2.5mm_P7.62mm_Horizontal, F.Cu at (203.5, 61.3)
- added R20: 4K7, Resistor_THT:R_Axial_DIN0207_L6.3mm_D2.5mm_P7.62mm_Horizontal, F.Cu at (203.5, 127.9)
- added R3: 4K7, Resistor_THT:R_Axial_DIN0207_L6.3mm_D2.5mm_P7.62mm_Horizontal, F.Cu at (203.5, 66.8)
- added R4: 4K7, Resistor_THT:R_Axial_DIN0207_L6.3mm_D2.5mm_P7.62mm_Horizontal, F.Cu at (203.5, 72.4)
- moved U1 2.80 mm to (113.1, 56.2)
Connections:
- U1 pad 10: unconnected-(U1-Pad10) -> /Z_CLOCK_IN
- U1 pad 11: GND -> Net-(R19-Pad2)
- U1 pad 12: unconnected-(U1-Pad12) -> /Z_DATA
- U1 pad 13: GND -> Net-(R20-Pad2)

Commit message: updates
Parts:
- added TB1: 2EDGR-2P, 2EDGK:2EDGR-2P, F.Cu at (71.1, 66.1)
- moved C1 140.0 mm to (276.9, 62.7)
- moved C10 140.0 mm to (276.9, 95.1)
- moved C2 140.0 mm to (276.9, 66.8)
- moved C4 140.0 mm to (276.9, 74.9)
- moved C5 140.0 mm to (276.9, 78.9)
- moved C7 140.0 mm to (276.9, 83.0)
- moved C8 140.0 mm to (276.9, 87.0)
- moved C9 140.0 mm to (276.9, 91.1)
- moved J1 127.9 mm to (116.7, 108.8), turned to 90 degrees
- moved J2 107.7 mm to (132.7, 108.8), turned to 90 degrees
- moved R2 99.3 mm to (113.7, 103.5), turned to 90 degrees
- moved R1 99.1 mm to (116.7, 103.5), turned to 90 degrees
- moved J4 88.0 mm to (148.7, 108.8), turned to 90 degrees
- moved R19 81.7 mm to (131.7, 83.5), turned to 90 degrees
- moved R20 80.2 mm to (136.7, 83.7), turned to 90 degrees
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Connections:
- R3 pad 2: Net-(U3-SENSOR_VP) -> /SEN_VP
- R4 pad 1: Net-(U3-SENSOR_VN) -> /SEN_VN
- U3 pad 10: unconnected-(U3-IO27-Pad10) -> /Y_CLOCK_OUT
- U3 pad 14: unconnected-(U3-GND-Pad14) -> GND
- U3 pad 15: unconnected-(U3-VIN-Pad15) -> +5V
- U3 pad 16: unconnected-(U3-3V3-Pad16) -> +3V3
- U3 pad 17: unconnected-(U3-GND-Pad17) -> GND
- U3 pad 2: unconnected-(U3-SENSOR_VP-Pad2) -> /SEN_VP
- U3 pad 20: unconnected-(U3-IO4-Pad20) -> /Y_DATA
- U3 pad 21: unconnected-(U3-IO16-Pad21) -> /Z_CLOCK_OUT
- U3 pad 22: unconnected-(U3-IO17-Pad22) -> /Z_DATA
- U3 pad 3: unconnected-(U3-SENSOR_VN-Pad3) -> /SEN_VN
- U3 pad 5: unconnected-(U3-IO35-Pad5) -> /Z_CLOCK_IN
- U3 pad 6: unconnected-(U3-IO32-Pad6) -> /Y_CLOCK_IN
- U3 pad 7: unconnected-(U3-IO33-Pad7) -> /X_CLOCK_IN
- U3 pad 8: unconnected-(U3-IO25-Pad8) -> /X_CLOCK_OUT
- U3 pad 9: unconnected-(U3-IO26-Pad9) -> /X_DATA

Commit message: updates
Parts:
- removed J3, J6: Conn_01x03, Connector_PinHeader_2.54mm:PinHeader_1x03_P2.54mm_Vertical
- moved C2 177.5 mm to (115.4, 140.2)
- moved C7 160.5 mm to (118.4, 58.0)
- moved C4 158.7 mm to (121.3, 106.0)
- moved C9 155.0 mm to (129.9, 140.2)
- moved C1 143.6 mm to (144.9, 119.2), turned to 90 degrees
- moved C10 139.1 mm to (145.4, 140.3)
- moved C5 128.1 mm to (159.9, 131.0)
- moved C8 126.4 mm to (159.9, 135.0)
- moved TB1 121.8 mm to (160.7, 148.6), turned to 90 degrees
- moved C11 108.9 mm to (119.6, 65.0)
- moved R12 104.9 mm to (112.9, 136.3), turned to 90 degrees
- moved JP3 102.6 mm to (140.3, 63.5)
- moved R11 99.1 mm to (123.4, 136.3), turned to 90 degrees
- moved JP1 98.5 mm to (135.3, 63.5)
- moved JP2 96.9 mm to (135.3, 104.0), turned to 180 degrees
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Connections:
- C10 pad 1: Net-(J4-VBUS) -> /SCALE_VIN
- C2 pad 1: Net-(J1-VBUS) -> /SCALE_VIN
- C9 pad 1: Net-(J2-VBUS) -> /SCALE_VIN
- J1 pad 1: Net-(J1-VBUS) -> /SCALE_VIN
- J2 pad 1: Net-(J2-VBUS) -> /SCALE_VIN
- J4 pad 1: Net-(J4-VBUS) -> /SCALE_VIN
- J5 pad 2: Net-(J1-VBUS) -> /SCALE_VIN
- R11 pad 2: Net-(J1-VBUS) -> /SCALE_VIN
- R12 pad 2: Net-(J1-VBUS) -> /SCALE_VIN
- R13 pad 2: Net-(J2-VBUS) -> /SCALE_VIN
- R14 pad 2: Net-(J2-VBUS) -> /SCALE_VIN
- R17 pad 2: Net-(J4-VBUS) -> /SCALE_VIN
- R18 pad 2: Net-(J4-VBUS) -> /SCALE_VIN
- TB1 pad 1: GND -> +5V
- TB1 pad 2: +5V -> GND
Other:
- board outline added: 60 x 100 mm

Commit message: new placement
Parts:
- removed J4: USB_B_Micro, MicroUSB-Breakout:MicroUSB
- added J20: Conn_01x03, Connector_PinHeader_2.54mm:PinHeader_1x03_P2.54mm_Vertical, F.Cu at (158.4, 129.5)
- added J3: USB_B_Micro, MicroUSB-Breakout:MicroUSB, F.Cu at (151.4, 145.2)
- added J6: Conn_01x01, MountingHole:MountingHole_3.5mm, F.Cu at (164.4, 59.0)
- added J7: Conn_01x01, MountingHole:MountingHole_3.5mm, F.Cu at (164.4, 135.0)
- added J8: Conn_01x01, MountingHole:MountingHole_3.5mm, F.Cu at (112.4, 135.0)
- J5: value Conn_01x03 -> Conn_01x01; footprint Connector_PinHeader_2.54mm:PinHeader_1x03_P2.54mm_Vertical -> MountingHole:MountingHole_3.5mm
- moved J5 88.0 mm to (112.4, 59.0)
- moved JP3 78.8 mm to (154.9, 141.0), turned to 90 degrees
- moved JP1 78.7 mm to (121.4, 141.0), turned to 90 degrees
- moved C7 56.9 mm to (159.9, 97.0), turned to 180 degrees
- moved C4 56.1 mm to (158.4, 64.0), turned to 180 degrees
- moved R3 52.4 mm to (116.6, 96.5), turned to 0 degrees
- moved R4 42.0 mm to (124.2, 100.0), turned to 180 degrees
- moved C11 38.9 mm to (157.9, 57.8), turned to 180 degrees
- moved JP2 37.2 mm to (138.7, 141.0), turned to 90 degrees
- moved U3 36.7 mm to (121.7, 80.5), turned to 90 degrees
- moved R12 11.2 mm to (117.6, 126.2), turned to 0 degrees
- moved R18 10.8 mm to (147.6, 126.0), turned to 0 degrees
- moved R14 10.4 mm to (132.1, 126.0), turned to 0 degrees
- moved U1 8.43 mm to (146.1, 107.0)
- moved C1 8.43 mm to (150.9, 113.3)
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Connections:
- JP1 pad 1: /Y_CLK -> /X_CLK
- JP1 pad 2: /Y_CLOCK_OUT -> /X_CLOCK_OUT
- JP2 pad 1: /Z_CLK -> /Y_CLK
- JP2 pad 2: /Z_CLOCK_OUT -> /Y_CLOCK_OUT
- JP3 pad 1: /X_CLK -> /Z_CLK
- JP3 pad 2: /X_CLOCK_OUT -> /Z_CLOCK_OUT

Commit message: updates
Parts:
- J5, J6, J7, J8: value Conn_01x01 -> MountingHole
- moved C5 66.4 mm to (141.9, 61.7), turned to 90 degrees
- moved J7 16.0 mm to (164.4, 119.0)
- moved J8 16.0 mm to (112.4, 119.0)
- moved U1 15.8 mm to (133.4, 116.5), turned to 90 degrees
- moved C4 12.1 mm to (146.6, 61.7), turned to 90 degrees
- moved R12 11.2 mm to (112.9, 136.3), turned to 90 degrees
- moved R14 10.5 mm to (129.9, 136.3), turned to 90 degrees
- moved R18 10.4 mm to (146.4, 136.3), turned to 90 degrees
- moved C8 9.40 mm to (161.9, 138.4)
- moved J20 7.63 mm to (164.4, 134.2)
- moved R19 5.52 mm to (156.9, 136.3)
- moved C11 5.51 mm to (153.3, 60.9), turned to 90 degrees
- moved R11 5.02 mm to (119.9, 136.3)
- moved R15 4.53 mm to (140.4, 136.3)
- moved C7 3.94 mm to (156.7, 94.7)
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Routing:
- net /SCALE_VIN: track 0.00 -> 157.3 mm
- net +3V3: track 0.00 -> 121.6 mm, vias 0 -> 1
- net /Z_CLOCK_OUT: track 0.00 -> 90.4 mm
- net /X_CLOCK_OUT: track 0.00 -> 77.0 mm
- net +5V: track 0.00 -> 73.6 mm, vias 0 -> 1
- net /Y_CLOCK_OUT: track 0.00 -> 68.5 mm
- net Net-(R19-Pad2): track 0.00 -> 67.4 mm
- net /Y_CLOCK_IN: track 0.00 -> 48.1 mm, vias 0 -> 1
- net /Y_DATA: track 0.00 -> 45.9 mm
- net Net-(R20-Pad2): track 0.00 -> 45.1 mm
- net /Z_CLOCK_IN: track 0.00 -> 44.9 mm, vias 0 -> 1
- net /Z_DATA: track 0.00 -> 44.9 mm
- net Net-(R2-Pad2): track 0.00 -> 38.9 mm
- net Net-(R15-Pad2): track 0.00 -> 34.5 mm
- net Net-(R16-Pad2): track 0.00 -> 32.5 mm
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- added copper zone on B.Cu, net GND
Other:
- board text added: "+"
