File: touchdro-board/touchdro-board.kicad_sch (KiCad schematic)
At the start: 2 parts, among them U1 74HC14, U2 DOIT-ESP32-DEVKIT-V1

Commit message: updates
Parts:
- removed U2: DOIT-ESP32-DEVKIT-V1, ESP32:ESP32-DOIT-DEVKIT, symbol ESP32:DOIT-ESP32-DEVKIT-V1
- added C1, C10, C2, C3, C4, C5, C7, C8, C9: 100n, symbol Device:C
- added C11, C6: 47u, symbol Device:C_Polarized
- added J1, J2, J4: USB_B_Micro, symbol Connector:USB_B_Micro
- added J3, J5, J6: Conn_01x03, symbol Connector_Generic:Conn_01x03
- added JP1, JP2, JP3: Jumper_2_Open, symbol Jumper:Jumper_2_Open
- added R1, R15, R16, R19, R2, R20, R3, R4: 4K7, symbol Device:R
- added R11, R12, R13, R14, R17, R18: 47K, symbol Device:R
- added U2: 74HC14, Package_DIP:DIP-14_W7.62mm, symbol 74xx:74HC14
- added U3: ESP32_DevKit_V1_DOIT, ESP32_DevKit_V1_DOIT:esp32_devkit_v1_doit, symbol ESP32-Devkit-V1:ESP32_DevKit_V1_DOIT
Connections:
- net Y_DATA: now reaches U1.8
- net Y_DATA: now also U3.20 (IO4)
- net at U1.9: now also R16.2
- net at U1.3: now also R2.2
- net X_DATA: now reaches U1.4
- net X_DATA: now also U3.9 (IO26)
- net Z_CLOCK_IN: now reaches U1.10
- net Z_CLOCK_IN: now also U3.5 (IO35)
- net at U1.11: now also R19.2
- net +3V3: now reaches U1.14 (VCC)
- net +3V3: now also C10.1, C11.1, C7.1, C8.1, C9.1, J3.3 (Pin_3), J5.3 (Pin_3), J6.3 (Pin_3), U2.14 (VCC), U3.16 (3V3)
- net GND: now reaches U1.7 (GND)
- net GND: now also C1.2, C10.2, C11.2, C2.2, C3.2, C4.2, C5.2, C6.2, C7.2, C8.2, C9.2, J1.5 (GND), J1.6 (Shield), J2.5 (GND), J2.6 (Shield), J4.5 (GND), J4.6 (Shield), R3.1, R4.2, U2.7 (GND), U3.14 (GND), U3.17 (GND)
- net at U1.1: now also R1.2
- net X_CLOCK_IN: now reaches U1.2
- net X_CLOCK_IN: now also U3.7 (IO33)
- net at U1.5: now also R15.2
- net Y_CLOCK_IN: now reaches U1.6
- net Y_CLOCK_IN: now also U3.6 (IO32)
- net Z_DATA: now reaches U1.12
- net Z_DATA: now also U3.22 (IO17)
- net at U1.13: now also R20.2
- new net: R3.2, U3.2 (SENSOR_VP)
- new net: C2.1, J1.1 (VBUS), J5.2 (Pin_2), R11.2, R12.2
- new net: C4.1, J4.1 (VBUS), J6.2 (Pin_2), R17.2, R18.2
- new net: C3.1, J2.1 (VBUS), J3.2 (Pin_2), R13.2, R14.2
- new net: R4.1, U3.3 (SENSOR_VN)
- new net +5V: C1.1, C5.1, C6.1, J3.1 (Pin_1), J5.1 (Pin_1), J6.1 (Pin_1), U3.15 (VIN)
- new net X_CLK: J1.3 (D+), JP3.1 (A), R1.1, R11.1
- new net X_CLOCK_OUT: JP3.2 (B), U3.8 (IO25)
- new net X_D: J1.2 (D-), R12.1, R2.1
- new net Y_CLK: J2.3 (D+), JP1.1 (A), R13.1, R15.1
- new net Y_CLOCK_OUT: JP1.2 (B), U3.10 (IO27)
- new net Y_D: J2.2 (D-), R14.1, R16.1
- new net Z_CLK: J4.3 (D+), JP2.1 (A), R17.1, R19.1
- new net Z_CLOCK_OUT: JP2.2 (B), U3.21 (IO16)
- new net Z_D: J4.2 (D-), R18.1, R20.1
- no-connect marks 0 -> 18
Other:
- moved on the sheet: U1A, U1B, U1G

Commit message: updates
Parts:
- removed C3: 100n, symbol Device:C
- removed U2: 74HC14, Package_DIP:DIP-14_W7.62mm, symbol 74xx:74HC14
- C1, C10, C2, C4, C5, C7, C8, C9: footprint (none) -> Capacitor_THT:C_Rect_L7.2mm_W3.0mm_P5.00mm_FKS2_FKP2_MKS2_MKP2; LCSC (none) -> C3034534
- C11, C6: footprint (none) -> Capacitor_THT:CP_Radial_D8.0mm_P3.50mm; LCSC (none) -> 03EC0571
- J1, J2, J4: footprint (none) -> MicroUSB-Breakout:MicroUSB
- J3, J5, J6: footprint (none) -> Connector_PinHeader_2.54mm:PinHeader_1x03_P2.54mm_Vertical
- JP1, JP2, JP3: footprint (none) -> Connector_PinHeader_2.54mm:PinHeader_1x02_P2.54mm_Vertical
- R1, R15, R16, R19, R2, R20, R3, R4: footprint (none) -> Resistor_THT:R_Axial_DIN0207_L6.3mm_D2.5mm_P7.62mm_Horizontal; LCSC (none) -> C119339
- R11, R12, R13, R14, R17, R18: footprint (none) -> Resistor_THT:R_Axial_DIN0207_L6.3mm_D2.5mm_P7.62mm_Horizontal; LCSC (none) -> C410613
- U1: LCSC (none) -> C2907
Connections:
- net +3V3: now also C1.1, C4.1, C5.1; no longer C10.1, C7.1, C8.1, C9.1
- net +5V: now also C7.1, C8.1; no longer C1.1, C5.1
- net at J4.1 (VBUS), J6.2 (Pin_2), R17.2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: now also C10.1; no longer C4.1
- net at J2.1 (VBUS), J3.2 (Pin_2), R13.2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: now also C9.1
Other:
- moved on the sheet: C11, C2, C6, J1, J2, J3, J4, J5, J6, JP1, JP2, JP3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

Commit message: updates
Parts:
- added TB1: 2EDGR-2P, 2EDGK:2EDGR-2P, symbol 2EDGK:2EDGR-2P
- U3: footprint ESP32_DevKit_V1_DOIT:esp32_devkit_v1_doit -> ESP32-Devkit-V1:esp32_devkit_v1_doit
Connections:
- net +5V: now also TB1.2
- net GND: now also TB1.1
- net SEN_VP: now reaches R3.2, U3.2 (SENSOR_VP)
- net SEN_VN: now reaches R4.1, U3.3 (SENSOR_VN)
Other:
- moved on the sheet: R3, R4

Commit message: updates
Parts:
- removed J3, J6: Conn_01x03, Connector_PinHeader_2.54mm:PinHeader_1x03_P2.54mm_Vertical, symbol Connector_Generic:Conn_01x03
Connections:
- net +5V: now also TB1.1; no longer TB1.2
- net GND: now also TB1.2; no longer TB1.1
- net SCALE_VIN: now reaches C2.1, J1.1 (VBUS), J5.2 (Pin_2), R11.2, R12.2
- net SCALE_VIN: now also C10.1, C9.1, J2.1 (VBUS), J4.1 (VBUS), R13.2, R14.2, R17.2, R18.2
Other:
- moved on the sheet: C1

Commit message: new placement
Parts:
- added J5, J6, J7, J8: Conn_01x01, MountingHole:MountingHole_3.5mm, symbol Connector_Generic:Conn_01x01
- renumbered J5 to J20, J4 to J3, JP3 to JP1, JP1 to JP2, JP2 to JP3
Connections:
- no-connect marks 18 -> 22

Commit message: updates
Parts:
- removed J5, J6, J7, J8: Conn_01x01, MountingHole:MountingHole_3.5mm, symbol Connector_Generic:Conn_01x01
- added J5, J6, J7, J8: MountingHole, MountingHole:MountingHole_3.5mm, symbol Mechanical:MountingHole
Connections:
- no-connect marks 22 -> 18
