File: touchdro-igaging/board/touchdro-igaging/touchdro-igaging.kicad_pcb (KiCad board)
At the start: 4 copper layers, 0 parts

Commit message: updates
Parts:
- added C35: 0603_100nF, Capacitors:C_0603, F.Cu at (180.5, 77.4)
- added C5: 0805_10uF, Capacitors:C_0805, F.Cu at (161.2, 115.5)
- added C6: 0603_100nF, Capacitors:C_0603, F.Cu at (156.9, 115.2)
- added C7: 0805_10uF, Capacitors:C_0805, F.Cu at (161.2, 118.5)
- added C8: 0603_100nF, Capacitors:C_0603, F.Cu at (156.9, 117.7)
- added G1: CE 8mm, Graphics:ce-8mm, F.Cu at (153.5, 79.3)
- added G2: Okimotus Logo, Graphics:okimotus-logo-20mm, F.Cu at (159.6, 73.1)
- added H10: Screw-3.2mm, Holes:ScrewHole-3.2mm, F.Cu at (145.3, 96.5)
- added H7: Screw-3.2mm, Holes:ScrewHole-3.2mm, F.Cu at (145.3, 73.9)
- added H8: Screw-3.2mm, Holes:ScrewHole-3.2mm, F.Cu at (145.3, 81.5)
- added H9: Screw-3.2mm, Holes:ScrewHole-3.2mm, F.Cu at (145.3, 89.0)
- added ISP1: AVR_ISP_8pin, Generic:AVR_ISP_8pin_VCC, F.Cu at (175.8, 82.1)
- added LED1: LED_TH_5mm_Green, Generic:LED_D5.0mm_Green, F.Cu at (172.5, 106.0)
- added LED2: LED_TH_5mm_Red, Generic:LED_D5.0mm_Red, F.Cu at (172.5, 113.2)
- added Q2: AO3400A, Commons:AO3400A, F.Cu at (182.6, 104.5)
- added Q3: AO3400A, Commons:AO3400A, F.Cu at (182.6, 109.0)
- added R3: 0603_100, Resistors:R_0603, F.Cu at (156.9, 120.2)
- added R47: 0603_4K7, Resistors:R_0603, F.Cu at (180.5, 79.9)
- added R48: 0603_100, Resistors:R_0603, F.Cu at (180.5, 82.5)
- added R49: 0603_100, Resistors:R_0603, F.Cu at (180.5, 85.0)
- added R56: 0603_470, Resistors:R_0603, F.Cu at (178.1, 103.6)
- added R57: 0603_10K, Resistors:R_0603, F.Cu at (178.1, 106.1)
- added R58: 0603_470, Resistors:R_0603, F.Cu at (178.1, 108.6)
- added R59: 0603_10K, Resistors:R_0603, F.Cu at (178.1, 111.1)
- added SW1: TS-1187A-B-A-B, Commons:TS-1187A-B-A-B, F.Cu at (176.4, 73.2)
- added U1: ATMEGA328PB-AU, Commons:ATMEGA328PB-AU, F.Cu at (161.0, 108.2)
- added U2: ~, Radio:HC05, F.Cu at (152.6, 104.7)
