File: touchdro-igaging/board/touchdro-igaging/touchdro-igaging.kicad_sch (KiCad schematic)
At the start: 7 parts, among them J1 UART, U1 ATMEGA328PB-AU

Commit message: updates
Parts:
- removed J1: UART, PinHeaders:PinHeader_1x03_P2.54mm, symbol Connector_Generic:Conn_01x03
- added U2: ~, Radio:HC05, symbol Radio:HC05
Connections:
- net LED_{1}: no longer U1.31 (TXD__[1]__PD1)
- net LED_{2}: no longer U1.30 (RXD__[0]__PD0)
- no-connect marks 3 -> 5
Changed lines of the file:
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@@
+	)
+	(no_connect
+		(at 214.63 57.15)
 	)
 	(no_connect
@@
 	)
 	(no_connect
+		(at 214.63 69.85)
+	)
+	(no_connect
 		(at 63.5 129.54)
 	)
@@
 	(wire
 		(pts
-			(xy 121.92 104.14) (xy 152.4 104.14)
-		)
-		(stroke
-			(width 0)
-			(type default)
-		)
-	)
-	(wire
-		(pts
 			(xy 41.91 73.66) (xy 41.91 76.2)
 		)
@@
 		(pts
 			(xy 121.92 93.98) (xy 140.97 93.98)
-		)
-		(stroke
-			(width 0)
-			(type default)
-		)
-	)
-	(wire
-		(pts
-			(xy 121.92 106.68) (xy 152.4 106.68)
 		)
 		(stroke
@@
 				(face "Bauhaus 93")
 				(size 30 30)
-			)
-			(justify left bottom)
-		)
-	)
-	(label "LED_{1}"
-		(at 140.97 106.68 0)
-		(fields_autoplaced yes)
-		(effects
-			(font
-				(size 1.27 1.27)
-			)
-			(justify left bottom)
-		)
-	)
-	(label "LED_{2}"
-		(at 140.97 104.14 0)
-		(fields_autoplaced yes)
-		(effects
-			(font
-				(size 1.27 1.27)
 			)
 			(justify left bottom)
@@
 		)
 		(instances
-			(project "board"
+			(project "touchdro-igaging"
 				(path "/65134029-dbd2-409a-85a8-13c2a33ff019"
 					(reference "#PWR051")
@@
 		)
 		(instances
-			(project "board"
+			(project "touchdro-igaging"
 				(path "/65134029-dbd2-409a-85a8-13c2a33ff019"
 					(reference "#PWR08")
@@
 		)
 		(instances
-			(project "board"
+			(project "touchdro-igaging"
 				(path "/65134029-dbd2-409a-85a8-13c2a33ff019"
 					(reference "#PWR05")
@@
 		)
 		(instances
-			(project "board"
+			(project "touchdro-igaging"
 				(path "/65134029-dbd2-409a-85a8-13c2a33ff019"
 					(reference "R3")
@@
 		)
 		(instances
-			(project "board"
+			(project "touchdro-igaging"
 				(path "/65134029-dbd2-409a-85a8-13c2a33ff019"
 					(reference "#PWR052")
@@
 		)
 		(instances
-			(project "board"
+			(project "touchdro-igaging"
 				(path "/65134029-dbd2-409a-85a8-13c2a33ff019"
 					(reference "C7")
@@
 		)
 		(instances
-			(project "board"
+			(project "touchdro-igaging"
 				(path "/65134029-dbd2-409a-85a8-13c2a33ff019"
 					(reference "C8")
-					(unit 1)
-				)
-			)
-		)
-	)
-	(symbol
-		(lib_id "Connector_Generic:Conn_01x03")
-		(at 157.48 104.14 0)
-		(unit 1)
-		(exclude_from_sim no)
-		(in_bom yes)
-		(on_board yes)
-		(dnp no)
-		(property "Reference" "J1"
-			(at 157.48 109.22 0)
-			(effects
-				(font
-					(size 1.27 1.27)
-				)
-			)
-		)
-		(property "Value" "UART"
-			(at 160.02 104.14 90)
-			(effects
-				(font
-					(size 1.27 1.27)
-				)
-			)
-		)
-		(property "Footprint" "PinHeaders:PinHeader_1x03_P2.54mm"
-			(at 157.48 104.14 0)
-			(effects
-				(font
-					(size 1.27 1.27)
-				)
-				(hide yes)
-			)
-		)
-		(property "Datasheet" ""
-			(at 157.48 104.14 0)
-			(effects
-				(font
-					(size 1.27 1.27)
-				)
-				(hide yes)
-			)
-		)
-		(property "Description" ""
-			(at 157.48 104.14 0)
-			(effects
-				(font
-					(size 1.27 1.27)
-				)
-				(hide yes)
-			)
-		)
-		(property "Type" "Virtual"
-			(at 157.48 104.14 0)
-			(effects
-				(font
-					(size 1.27 1.27)
-				)
-				(hide yes)
-			)
-		)
-		(pin "1"
-		)
-		(pin "2"
-		)
-		(pin "3"
-		)
-		(instances
-			(project "board"
-				(path "/65134029-dbd2-409a-85a8-13c2a33ff019"
-					(reference "J1")
-					(unit 1)
-				)
-			)
-		)
-	)
-	(symbol
-		(lib_id "power:GND")
-		(at 152.4 101.6 270)
-		(unit 1)
-		(exclude_from_sim no)
-		(in_bom yes)
-		(on_board yes)
-		(dnp no)
-		(property "Reference" "#PWR012"
-			(at 146.05 101.6 0)
-			(effects
-				(font
-					(size 1.27 1.27)
-				)
-				(hide yes)
-			)
-		)
-		(property "Value" "GND"
-			(at 148.59 101.6 0)
-			(effects
-				(font
-					(size 1.27 1.27)
-				)
-				(hide yes)
-			)
-		)
-		(property "Footprint" ""
-			(at 152.4 101.6 0)
-			(effects
-				(font
-					(size 1.27 1.27)
-				)
-				(hide yes)
-			)
-		)
-		(property "Datasheet" ""
-			(at 152.4 101.6 0)
-			(effects
-				(font
-					(size 1.27 1.27)
-				)
-				(hide yes)
-			)
-		)
-		(property "Description" ""
-			(at 152.4 101.6 0)
-			(effects
-				(font
-					(size 1.27 1.27)
-				)
-				(hide yes)
-			)
-		)
-		(pin "1"
-		)
-		(instances
-			(project "board"
-				(path "/65134029-dbd2-409a-85a8-13c2a33ff019"
-					(reference "#PWR012")
 					(unit 1)
 				)
@@
 		)
 		(instances
-			(project "board"
+			(project "touchdro-igaging"
 				(path "/65134029-dbd2-409a-85a8-13c2a33ff019"
 					(reference "#PWR06")
@@
 		)
 		(instances
-			(project "board"
+			(project "touchdro-igaging"
 				(path "/65134029-dbd2-409a-85a8-13c2a33ff019"
 					(reference "C6")
@@
 		)
 		(instances
-			(project "board"
+			(project "touchdro-igaging"
 				(path "/65134029-dbd2-409a-85a8-13c2a33ff019"
 					(reference "#PWR010")
@@
 		)
 		(instances
-			(project "board"
+			(project "touchdro-igaging"
 				(path "/65134029-dbd2-409a-85a8-13c2a33ff019"
 					(reference "C5")
@@
 		)
 		(instances
-			(project "board"
+			(project "touchdro-igaging"
 				(path "/65134029-dbd2-409a-85a8-13c2a33ff019"
 					(reference "U1")
+					(unit 1)
+				)
+			)
+		)
+	)
+	(symbol
+		(lib_id "Radio:HC05")
+		(at 223.52 63.5 0)
+		(unit 1)
+		(exclude_from_sim no)
+		(in_bom yes)
+		(on_board yes)
+		(dnp no)
+		(property "Reference" "U2"
+			(at 222.758 53.086 0)
+			(effects
+				(font
+					(size 1.27 1.27)
+				)
+				(justify left)
+			)
+		)
+		(property "Value" "~"
+			(at 232.41 64.77 0)
+			(effects
+				(font
+					(size 1.27 1.27)
+				)
+				(justify left)
+			)
+		)
+		(property "Footprint" "Radio:HC05"
+			(at 215.9 53.34 0)
+			(effects
+				(font
+					(size 1.27 1.27)
+				)
+				(hide yes)
+			)
+		)
+		(property "Datasheet" ""
+			(at 215.9 53.34 0)
+			(effects
+				(font
+					(size 1.27 1.27)
+				)
+				(hide yes)
+			)
+		)
+		(property "Description" "HC05"
+			(at 215.9 53.34 0)
+			(effects
+				(font
+					(size 1.27 1.27)
+				)
+				(hide yes)
+			)
+		)
+		(pin "1"
+		)
+		(pin "2"
+		)
+		(pin "4"
+		)
+		(pin "5"
+		)
+		(pin "3"
+		)
+		(pin "6"
+		)
+		(instances
+			(project "touchdro-igaging"
+				(path "/65134029-dbd2-409a-85a8-13c2a33ff019"
+					(reference "U2")
 					(unit 1)
 				)
@@
 		)
 		(instances
-			(project "board"
+			(project "touchdro-igaging"
 				(path "/65134029-dbd2-409a-85a8-13c2a33ff019"
 					(reference "#PWR021")
@@
 		)
 		(instances
-			(project "board"
+			(project "touchdro-igaging"
 				(path "/65134029-dbd2-409a-85a8-13c2a33ff019"
 					(reference "#PWR011")
@@
 		)
 		(instances
-			(project "board"
+			(project "touchdro-igaging"
 				(path "/65134029-dbd2-409a-85a8-13c2a33ff019"
 					(page "6")
@@
 		)
 		(instances
-			(project "board"
+			(project "touchdro-igaging"
 				(path "/65134029-dbd2-409a-85a8-13c2a33ff019"
 					(page "8")
@@
 		)
 		(instances
-			(project "board"
+			(project "touchdro-igaging"
 				(path "/65134029-dbd2-409a-85a8-13c2a33ff019"
 					(page "9")
